File: hw/msp430_servo.sch (KiCad schematic (older format))
At the start: 45 parts, among them IC1 MSP430G2553IPW20, IC2 L78L33ACUTR, P1 CONN_01X02, P10 CONN_01X03, P2 CONN_01X01, P3 CONN_01X03, P4 CONN_01X03, P5 CONN_01X02, P6 CONN_01X02, P7 CONN_01X02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

Commit message: silk repair, assembly
Parts:
- C1, C2, C3, C4, C5, C6, C7, C8, C9: symbol C_Small -> Device:C_Small
- D1: symbol UniTSV -> msp430_servo-rescue:UniTSV
- D2: symbol D_Schottky_x2_KCom_AAK -> Device:D_Schottky_x2_KCom_AAK
- IC1: symbol MSP430G2553IPW20 -> my_texas:MSP430G2553IPW20
- IC2: symbol MC78L05ACH -> msp430_servo-rescue:MC78L05ACH
- LED1, LED2: symbol Led_Small -> msp430_servo-rescue:Led_Small
- P1, P5, P6, P7, P8: symbol CONN_01X02 -> msp430_servo-rescue:CONN_01X02
- P10, P3, P4, P9: symbol CONN_01X03 -> msp430_servo-rescue:CONN_01X03
- P2: symbol CONN_01X01 -> msp430_servo-rescue:CONN_01X01
- Q1, Q2: symbol BC817-40 -> msp430_servo-rescue:BC817-40
- R1, R10, R11, R12, R13, R14, R15, R16, R17, R18, R2, R3, R4, R5, R6, R7, R8, R9: symbol R_Small -> Device:R_Small
